File: hardware/featherbyte-uno-v1.0.0/featherbyte-uno-v1.0.0.kicad_pcb (KiCad board)
At the start: 2 copper layers, 54 x 60 mm, 63 parts, among them J1 Conn_01x08, J10 Conn_01x09, J2 Conn_01x10, J3 Conn_01x06, J5 USB_C_Receptacle_16P, J6 SWD Connector, J7 Terminal Block, J8 USB_C_Receptacle_16P, J9 BOOT1, SW1 Reset, SW2 BOOT0, SW3 SW_DIP_x04, U1 CH32V203CxT6, U2 TJA1050, U4 AMS1117-3.3, U5 USBLC6-2P6, U6 USBLC6-2P6, Y1 8M, Y3 32.768K

Commit message: routing process ongoing
Parts:
- removed R11, R12: 0R, Resistor_SMD:R_0603_1608Metric
- moved D4 43.4 mm to (85.6, 75.7), turned to -90 degrees
- moved R14 42.3 mm to (89.9, 77.7), turned to 135 degrees
- moved C15 28.9 mm to (77.4, 109.1), turned to 90 degrees
- moved SW1 27.4 mm to (83.8, 113.4)
- moved SW2 27.4 mm to (111.2, 113.4)
- moved R8 27.3 mm to (79.0, 109.1), turned to 90 degrees
- moved J9 19.2 mm to (107.8, 94.7), turned to -135 degrees
- moved R9 17.6 mm to (105.9, 109.1)
- moved C16 17.6 mm to (104.2, 109.1)
- moved TP1 10.8 mm to (86.1, 69.4)
- moved R10 4.28 mm to (83.1, 82.1), turned to -135 degrees
- moved C14 3.05 mm to (87.2, 82.8), turned to 135 degrees
- moved C11 2.10 mm to (96.0, 78.2)
- moved J6 1.36 mm to (75.0, 72.5)
- moved C12 0.40 mm to (88.3, 81.7)
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Connections:
- J2 pad 3: /VREF -> unconnected-(J2-Pin_3-Pad3)
- U1 pad 16: unconnected-(U1-PA6/ADC6-Pad16) -> /D2
- U1 pad 17: unconnected-(U1-PA7/ADC7-Pad17) -> /D3
- U1 pad 29: unconnected-(U1-PA8-Pad29) -> /D4
- U1 pad 30: unconnected-(U1-PA9-Pad30) -> /D5
- U1 pad 31: unconnected-(U1-PA10-Pad31) -> /D6
- U1 pad 38: unconnected-(U1-PA15-Pad38) -> /D7
- U1 pad 39: unconnected-(U1-PB3-Pad39) -> /D8
- U1 pad 40: unconnected-(U1-PB4-Pad40) -> /D9
- U1 pad 41: unconnected-(U1-PB5-Pad41) -> /LED
Routing:
- net /NRST: track 0.00 -> 83.6 mm, vias 0 -> 1
- net /BOOT0: track 0.00 -> 45.4 mm, vias 0 -> 2
- net /D7: track 0.00 -> 36.3 mm, vias 0 -> 1
- net /D9: track 0.00 -> 36.1 mm, vias 0 -> 1
- net /D8: track 0.00 -> 35.4 mm, vias 0 -> 1
- net /D4: track 0.00 -> 33.3 mm, vias 0 -> 1
- net /D5: track 0.00 -> 33.2 mm, vias 0 -> 1
- net /D6: track 0.00 -> 31.3 mm, vias 0 -> 1
- net /D2: track 0.00 -> 30.3 mm, vias 0 -> 1
- net /SWDIO: track 0.00 -> 29.3 mm, vias 0 -> 1
- net /D3: track 0.00 -> 28.7 mm, vias 0 -> 1
- net /CAN0TX: track 0.00 -> 22.1 mm, vias 0 -> 2
- net /USBHD_DP: track 0.00 -> 19.5 mm
- net /USBHD_DN: track 0.00 -> 19.2 mm
- net /USBD_DN: track 0.00 -> 19.0 mm
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
Commit message: all pins routed
Parts:
- added JP2: Jumper, Jumper:SolderJumper-2_P1.3mm_Open_TrianglePad1.0x1.5mm, B.Cu at (104.1, 87.6)
- added JP3: Jumper2, Jumper:SolderJumper-2_P1.3mm_Open_TrianglePad1.0x1.5mm, B.Cu at (102.3, 89.4)
- moved J9 5.69 mm to (109.1, 89.2), turned to -45 degrees
- moved D1 1.95 mm to (89.8, 65.4)
- moved D2 0.83 mm to (105.0, 67.1)
- moved TP1 0.23 mm to (86.2, 69.2)
Connections:
- U1 pad 21: unconnected-(U1-PB10-Pad21) -> /SCL
- U1 pad 22: unconnected-(U1-PB11-Pad22) -> /SDA
Routing:
- net /SCL: track 0.00 -> 46.1 mm, vias 0 -> 2
- net /SDA: track 0.00 -> 39.0 mm, vias 0 -> 2
- net /A4: track 37.8 -> 50.2 mm, vias 0 -> 1
- net /A5: track 40.9 -> 49.8 mm, vias 0 -> 1
- net +3.3V: track 12.5 -> 9.14 mm
- net /D5: track 33.2 -> 31.8 mm
- net /BOOT1: track 9.70 -> 10.9 mm, vias 0 -> 1
- net /CAN0RX: track 18.0 -> 18.6 mm

Commit message: all routing done
Parts:
- moved R2 2.05 mm to (117.7, 58.0)
- moved R3 2.05 mm to (117.7, 59.6)
- moved C11 1.02 mm to (95.0, 78.4), turned to 135 degrees
- moved R15 0.77 mm to (100.2, 62.8)
- moved R16 0.77 mm to (100.2, 57.6)
- moved R5 0.77 mm to (100.2, 59.3)
- moved R6 0.77 mm to (100.2, 61.0)
- moved SW3 0.77 mm to (93.3, 60.2)
- moved D1 0.29 mm to (89.5, 65.3)
- moved TP1 0.16 mm to (86.3, 69.3)
- moved JP2 0.14 mm to (104.2, 87.7)
- moved JP3 0.12 mm to (102.4, 89.5)
- moved TP2 0.09 mm to (96.8, 66.8)
Connections:
- J6 pad 6: unconnected-(J6-Pin_6-Pad6) -> GND
Routing:
- net +3.3V: track 9.14 -> 190.0 mm, vias 0 -> 10
- net +5V: track 4.86 -> 84.9 mm, vias 0 -> 4
- net VBUS: track 0.00 -> 41.5 mm
- net /VBUS1: track 0.00 -> 33.9 mm
- net /VBUS2: track 0.00 -> 33.4 mm
- net GND: track 0.00 -> 6.90 mm, vias 0 -> 92
- net Net-(J5-CC1): track 9.92 -> 13.7 mm, vias 0 -> 2
- net /USBD_D-: track 5.09 -> 7.89 mm
- net /USBD_D+: track 5.09 -> 7.35 mm
- net Net-(J8-CC1): track 7.44 -> 9.68 mm, vias 0 -> 2
- net Net-(J8-CC2): track 10.9 -> 12.9 mm, vias 0 -> 2
- net /BOOT0: track 45.4 -> 46.9 mm
- net /D7: track 36.3 -> 37.7 mm
- net Net-(J5-CC2): track 15.3 -> 14.2 mm
- net /SDA: track 39.0 -> 40.1 mm
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- added copper zone on F.Cu, net +3.3V
- added copper zone on F.Cu, net +5V
- added copper zone on B.Cu, net GND
- added copper zone on F.Cu, net GND
